File: hardware/bastwan-wle.kicad_pcb (KiCad board)
At the start: 2 copper layers, 0 parts

Commit message: Add_footprin_Rak
Parts:
- added D1: PGB1010402KR, Inductor_SMD:L_0402_1005Metric, F.Cu at (127.8, 69.4)
- added D2: MBR120, Diode_SMD:D_SOD-123, F.Cu at (133.9, 47.9)
- added D4: CHR, LED_SMD:LED_0805_2012Metric_Pad1.15x1.40mm_HandSolder, F.Cu at (139.1, 31.0)
- added D5: D13, LED_SMD:LED_0805_2012Metric_Pad1.15x1.40mm_HandSolder, F.Cu at (145.1, 38.9)
- added J1: USB_B_Micro, Connectors:U254051N4BH806, F.Cu at (116.3, 74.0)
- added J2: Conn_Right, Connector_PinSocket_2.54mm:PinSocket_1x12_P2.54mm_Vertical, F.Cu at (130.4, 63.9)
- added J3: Conn_Left, Connector_PinSocket_2.54mm:PinSocket_1x16_P2.54mm_Vertical, F.Cu at (120.2, 84.2)
- added J5: SWD, Connector_PinHeader_2.54mm:PinHeader_1x04_P2.54mm_Vertical, F.Cu at (127.0, 80.3)
- added Q1: DMG3415U-7, Package_TO_SOT_SMD:SOT-23, F.Cu at (137.5, 52.5)
- added REF**: MountingHole_2.7mm_M2.5, MountingHole:MountingHole_2.7mm_M2.5, F.Cu at (162.2, 65.2)
- added REF**: MountingHole_2.7mm_M2.5, MountingHole:MountingHole_2.7mm_M2.5, F.Cu at (162.2, 83.0)
- added REF**: MountingHole_2.7mm_M2.5, MountingHole:MountingHole_2.7mm_M2.5, F.Cu at (116.4, 83.0)
- added REF**: MountingHole_2.7mm_M2.5, MountingHole:MountingHole_2.7mm_M2.5, F.Cu at (116.4, 65.2)
- added SW1: RST, Button_Switch_SMD:SW_SPST_TL3342, F.Cu at (139.7, 77.5)
- added U1: RAK3172, ElectronicCats-KiCad-Libraries:RAK3172, F.Cu at (159.9, 66.3)
- added U2: AP2112K-3.3TRG1, Package_TO_SOT_SMD:TSOT-23-5, F.Cu at (145.7, 47.6)
- added U3: CH340C, Package_SO:SOIC-16_3.9x9.9mm_P1.27mm, F.Cu at (163.2, 31.9)
- added U5: MCP73831-3-OT, Package_TO_SOT_SMD:SOT-23-5, F.Cu at (134.8, 39.1)
Other:
- board outline added: 50.8 x 22.9 mm
- net class Default: trace_width 0.2 -> 0.25; via_dia 0.6 -> 0.8; via_drill 0.3 -> 0.4
- rule pad_to_mask_clearance: 0 -> 0.051
- rule trace_min: 0.1524 -> 0.2
- rule via_min_size: 0.6 -> 0.4
- board text added: "3V3"
- board text added: "A0"
- board text added: "A1"
- board text added: "A2"
- board text added: "A3"
- board text added: "A4"
- board text added: "A5"
- board text added: "AREF"
- board text added: "EN"
- board text added: "F0"
- board text added: "F1"
- board text added: "F2"
- board text added: "F3"
- board text added: "F4"
- board text added: "F5"
- board text added: "F6"
- board text added: "FREE"
- board text added: "GND"
- board text added: "MISO"
- board text added: "MOSI"
- board text added: "RX"
- board text added: "SCK"
- board text added: "SCL"
- board text added: "SDA"
- board text added: "TX"
- board text added: "VBAT"
- board text added: "VUSB"
- board text added: "~RST"

Commit message: Route
Parts:
- added AE1: Antenna, Rf:SMA_EDGE, F.Cu at (164.5, 74.2)
- added C2: 47pF, Capacitor_SMD:C_0402_1005Metric_Pad0.74x0.62mm_HandSolder, F.Cu at (160.3, 69.2)
- added C3: 10uF, Capacitor_SMD:C_0402_1005Metric_Pad0.74x0.62mm_HandSolder, F.Cu at (134.7, 70.0)
- added C4: 10uF, Capacitor_SMD:C_0402_1005Metric_Pad0.74x0.62mm_HandSolder, F.Cu at (137.0, 70.0)
- added C5: 10uF, Capacitor_SMD:C_0402_1005Metric_Pad0.74x0.62mm_HandSolder, F.Cu at (127.3, 66.2)
- added R1: 100K, Resistor_SMD:R_0402_1005Metric_Pad0.72x0.64mm_HandSolder, F.Cu at (127.3, 72.8)
- added R2: 100K, Resistor_SMD:R_0402_1005Metric_Pad0.72x0.64mm_HandSolder, F.Cu at (126.7, 71.2)
- added R3: 1M, Resistor_SMD:R_0402_1005Metric_Pad0.72x0.64mm_HandSolder, F.Cu at (131.8, 76.8)
- added R4: 1.5M, Resistor_SMD:R_0402_1005Metric_Pad0.72x0.64mm_HandSolder, F.Cu at (131.8, 79.0)
- added R6: 1K, Resistor_SMD:R_0402_1005Metric_Pad0.72x0.64mm_HandSolder, F.Cu at (129.5, 66.2)
- added R8: 330, Resistor_SMD:R_0402_1005Metric_Pad0.72x0.64mm_HandSolder, F.Cu at (125.8, 69.2)
- added R9: 330, Resistor_SMD:R_0402_1005Metric_Pad0.72x0.64mm_HandSolder, F.Cu at (141.0, 71.2)
- D4, D5: footprint LED_SMD:LED_0805_2012Metric_Pad1.15x1.40mm_HandSolder -> LED_SMD:LED_0603_1608Metric_Pad1.05x0.95mm_HandSolder
- U1: footprint ElectronicCats-KiCad-Libraries:RAK3172 -> Rf:RAK3172
- moved U3 59.2 mm to (126.1, 78.0)
- moved D4 43.9 mm to (123.4, 72.0)
- moved D1 34.9 mm to (162.7, 69.2), turned to 270 degrees
- moved U5 30.2 mm to (128.2, 68.6)
- moved D5 29.7 mm to (141.0, 68.3), turned to 90 degrees
- moved U2 29.3 mm to (130.2, 72.5)
- moved D2 20.2 mm to (135.9, 68.0), turned to 180 degrees
- moved Q1 17.1 mm to (131.8, 68.6), turned to 180 degrees
- moved U1 16.9 mm to (143.0, 66.5), turned to 0 degrees
- moved J5 10.5 mm to (134.2, 72.7), turned to 0 degrees
- moved SW1 0.69 mm to (139.1, 77.6)
Routing:
- net /A0: track 0.00 -> 52.2 mm, vias 0 -> 1
- net /A1: track 0.00 -> 34.9 mm, vias 0 -> 2
- net VBUS: track 0.00 -> 29.6 mm
- net /A2: track 0.00 -> 27.9 mm, vias 0 -> 1
- net /D12: track 0.00 -> 27.9 mm, vias 0 -> 2
- net /D13: track 0.00 -> 27.8 mm, vias 0 -> 1
- net /D11: track 0.00 -> 23.7 mm, vias 0 -> 1
- net /A3: track 0.00 -> 23.0 mm, vias 0 -> 1
- net /TX: track 0.00 -> 22.8 mm
- net /A4: track 0.00 -> 22.6 mm, vias 0 -> 2
- net /RX: track 0.00 -> 21.1 mm
- net /EN: track 0.00 -> 19.7 mm, vias 0 -> 2
- net /D9: track 0.00 -> 18.9 mm, vias 0 -> 1
- net /D6: track 0.00 -> 15.0 mm, vias 0 -> 1
- net /D-: track 0.00 -> 14.6 mm
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- added copper zone on B.Cu, net GND
- added copper zone on F.Cu, net GND

Commit message: Add_connector
Parts:
- AE1: footprint Rf:SMA_EDGE -> Connectors:JST_S2B-PH-SM4-TB(LF)(SN)
- SW1: footprint Button_Switch_SMD:SW_SPST_TL3342 -> Switches:C455281
- U3: moved to B.Cu
- moved AE1 40.5 mm to (124.2, 70.3)
- moved D2 17.1 mm to (121.3, 77.0), turned to 90 degrees
- moved U1 15.2 mm to (158.2, 66.2), turned to 270 degrees
- moved C3 13.9 mm to (123.0, 77.5), turned to 270 degrees
- moved C4 10.6 mm to (129.4, 77.3), turned to 270 degrees
- moved SW1 8.66 mm to (130.4, 76.8), turned to 0 degrees
- moved Q1 8.39 mm to (125.6, 74.2)
- moved J5 8.14 mm to (138.6, 79.6), turned to 180 degrees
- moved C5 6.93 mm to (130.4, 72.4)
- moved U2 6.27 mm to (126.7, 77.7)
- moved R1 5.78 mm to (123.9, 77.5)
- moved R6 5.51 mm to (133.7, 69.8), turned to 270 degrees
- moved D4 5.39 mm to (128.5, 73.7)
- moved R2 5.29 mm to (123.0, 75.0), turned to 90 degrees
- moved U3 4.00 mm to (126.2, 74.0), turned to 0 degrees
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Routing:
- net /A0: track 52.2 -> 0.00 mm, vias 1 -> 0
- net /A1: track 34.9 -> 0.00 mm, vias 2 -> 0
- net VBUS: track 29.6 -> 0.00 mm
- net /A2: track 27.9 -> 0.00 mm, vias 1 -> 0
- net /D12: track 27.9 -> 0.00 mm, vias 2 -> 0
- net /D13: track 27.8 -> 0.00 mm, vias 1 -> 0
- net /D11: track 23.7 -> 0.00 mm, vias 1 -> 0
- net /A3: track 23.0 -> 0.00 mm, vias 1 -> 0
- net /TX: track 22.8 -> 0.00 mm
- net /A4: track 22.6 -> 0.00 mm, vias 2 -> 0
- net /RX: track 21.1 -> 0.00 mm
- net /EN: track 19.7 -> 0.00 mm, vias 2 -> 0
- net /D9: track 18.9 -> 3.69 mm, vias 1 -> 0
- net /D6: track 15.0 -> 0.00 mm, vias 1 -> 0
- net +BATT: track 14.6 -> 0.00 mm
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- removed copper zone on B.Cu, net GND
- removed copper zone on F.Cu, net GND

Commit message: change to cp2102
Parts:
- removed U3: CH340C, Package_SO:SOIC-16_3.9x9.9mm_P1.27mm
Other:
- board text added: "B0"
- board text added: "D10"
- board text added: "D11"
- board text added: "D12"
- board text added: "D13"
- board text added: "D5"
- board text added: "D6"
- board text added: "D9"
- board text added: "NC"
- board text removed: "A5"
- board text removed: "F0"
- board text removed: "F1"
- board text removed: "F2"
- board text removed: "F3"
- board text removed: "F4"
- board text removed: "F5"
- board text removed: "F6"
- board text removed: "FREE"

Commit message: New_route
Parts:
- added C1: 0.1uF, Capacitor_SMD:C_0402_1005Metric_Pad0.74x0.62mm_HandSolder, B.Cu at (127.7, 75.0)
- added C6: 0.1uF, Capacitor_SMD:C_0402_1005Metric_Pad0.74x0.62mm_HandSolder, F.Cu at (140.8, 77.8)
- added J4: Conn_Battery, Connectors:JST_S2B-PH-SM4-TB(LF)(SN), F.Cu at (123.3, 70.0)
- added U3: CP2102N-A01-GQFN28, Package_DFN_QFN:QFN-28-1EP_5x5mm_P0.5mm_EP3.35x3.35mm, B.Cu at (131.7, 73.7)
- AE1: footprint Connectors:JST_S2B-PH-SM4-TB(LF)(SN) -> agroin:SMA_EDGE
- moved AE1 40.4 mm to (164.5, 73.7)
- moved C2 9.36 mm to (161.1, 78.5), turned to 90 degrees
- moved D1 9.25 mm to (163.0, 78.4), turned to 90 degrees
- moved D2 0.83 mm to (121.4, 77.8)
- moved R8 0.72 mm to (128.1, 70.9)
- moved J5 0.57 mm to (138.1, 79.4)
- moved D4 0.46 mm to (128.1, 73.8)
- turned Q1 to 0 degrees
Routing:
- net GND: track 0.00 -> 95.5 mm, vias 0 -> 10
- net /A0: track 0.00 -> 49.1 mm, vias 0 -> 1
- net VBUS: track 0.00 -> 41.9 mm, vias 0 -> 1
- net +BATT: track 0.00 -> 41.1 mm, vias 0 -> 1
- net +3V3: track 0.00 -> 40.4 mm, vias 0 -> 2
- net /A4: track 0.00 -> 39.1 mm, vias 0 -> 1
- net /RST: track 0.00 -> 35.2 mm, vias 0 -> 2
- net /EN: track 0.00 -> 34.2 mm, vias 0 -> 2
- net /TX_USB: track 0.00 -> 32.3 mm, vias 0 -> 1
- net /RX_USB: track 0.00 -> 31.7 mm, vias 0 -> 1
- net /D11: track 0.00 -> 25.7 mm, vias 0 -> 1
- net /D10: track 0.00 -> 23.9 mm, vias 0 -> 1
- net /D12: track 0.00 -> 22.4 mm
- net /SWDIO: track 0.00 -> 22.2 mm, vias 0 -> 2
- net /BOOT0: track 0.00 -> 21.6 mm, vias 0 -> 1
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- added copper zone on B.Cu, net GND
- added copper zone on F.Cu, net GND

Commit message: Add_Logo
Parts:
- added G***: LOGO, Aesthetics:bast_8x8, B.Cu at (150.9, 73.8)
- renumbered SW1 to RST
