File: hardware/bastwan-wle.sch (KiCad schematic (older format))
At the start: 29 parts, among them J1 USB_B_Micro, J2 Conn_Right, J3 Conn_Left, J4 Conn_Battery, J5 SWD, Q1 DMG3415U-7, SW1 RST, U1 RAK3172, U2 MCP1700-1202E_SOT23, U3 CP2102N-A01-GQFN28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

Commit message: Last_route
Parts:
- removed U2: MCP1700-1202E_SOT23, Package_TO_SOT_SMD:SOT-23, symbol Regulator_Linear:MCP1700-1202E_SOT23
- added U2: MCP1700_DFN6, Package_DFN_QFN:DFN-6-1EP_2x2mm_P0.65mm_EP1x1.6mm, symbol Regulator:MCP1700_DFN6
Changed lines of the file:
@@
 Wire Notes Line
 	4935 8055 4920 8055
-$Comp
-L Regulator_Linear:MCP1700-1202E_SOT23 U2
-U 1 1 60F17AD5
-P 2985 4295
-F 0 "U2" H 2985 4537 50  0000 C CNN
-F 1 "MCP1700-1202E_SOT23" H 2985 4446 50  0000 C CNN
-F 2 "Package_TO_SOT_SMD:SOT-23" H 2985 4520 50  0001 C CNN
-F 3 "http://ww1.microchip.com/downloads/en/DeviceDoc/20001826D.pdf" H 2985 4295 50  0001 C CNN
-	1    2985 4295
-	1    0    0    -1
-$EndComp
 Wire Wire Line
 	2985 4595 2985 4685
@@
 	2240 4295 2685 4295
 NoConn ~ 3950 1425
+$Comp
+L Regulator:MCP1700_DFN6 U2
+U 1 1 60F6422D
+P 2985 4295
+F 0 "U2" H 2985 4537 50  0000 C CNN
+F 1 "MCP1700_DFN6" H 2985 4446 50  0000 C CNN
+F 2 "Package_DFN_QFN:DFN-6-1EP_2x2mm_P0.65mm_EP1x1.6mm" H 2985 4520 50  0001 C CNN
+F 3 "http://ww1.microchip.com/downloads/en/DeviceDoc/20001826D.pdf" H 2985 4295 50  0001 C CNN
+	1    2985 4295
+	1    0    0    -1
+$EndComp
 $EndSCHEMATC

Commit message: Add_BOM_Change_footprint
Parts:
- AE1: #LCSC (none) -> C1509219; Proveedor (none) -> LCSC; manf# - -> HJ-SMA023
- C1, C6: #LCSC (none) -> C106209; Proveedor (none) -> LCSC; manf# (none) -> CC0402ZRY5V7BB104
- C2: footprint Capacitor_SMD:C_0402_1005Metric_Pad0.74x0.62mm_HandSolder -> Capacitor_SMD:C_0603_1608Metric_Pad1.08x0.95mm_HandSolder; #LCSC (none) -> C519486; Proveedor (none) -> LCSC; manf# 0603CG470J500NT -> CC0603FRNPO9BN470
- C3, C4, C5: #LCSC (none) -> C15525; Proveedor (none) -> LCSC; manf# GRM188R61C106MA73D -> CL05A106MQ5NUNC
- C7: footprint (none) -> Capacitor_SMD:C_0402_1005Metric_Pad0.74x0.62mm_HandSolder; #LCSC (none) -> C107372; Proveedor (none) -> LCSC; manf# (none) -> CL05A105KQ5NNNC
- D1: #LCSC (none) -> C10676; Proveedor (none) -> LCSC
- D2: #LCSC (none) -> C130880; Proveedor (none) -> LCSC
- D4: #LCSC (none) -> C72043; Proveedor (none) -> LCSC; manf# NCD0805G1 -> 19-217/GHC-YR1S2/3T
- D5: #LCSC (none) -> C72044; Proveedor (none) -> LCSC; manf# BL-HB335A-TRE -> 19-217/R6C-AL1M2VY/3T
- J1: #LCSC (none) -> C319170; Proveedor (none) -> LCSC
- J4: #LCSC (none) -> C295747; Proveedor (none) -> LCSC; manf# - -> S2B-PH-SM4-TB(LF)(SN)
- Q1: #LCSC (none) -> C459537; Proveedor (none) -> LCSC
- R2: #LCSC (none) -> C284273; Proveedor (none) -> LCSC; manf# RC0603FR-07100KL -> ARG02FTC1003
- R3: #LCSC (none) -> C93949; Proveedor (none) -> LCSC; manf# RC0603JR-071ML -> RC0402JR-071ML
- R4: #LCSC (none) -> C22276; Proveedor (none) -> LCSC; manf# RC0603JR-071M5L -> 0402WGF1504TCE
- R6: #LCSC (none) -> C425517; Proveedor (none) -> LCSC; manf# RC0603JR-071KL -> TC0250F1001TCE
- R8, R9: #LCSC (none) -> C105876; Proveedor (none) -> LCSC; manf# RC0603FR-07330RL -> RC0402JR-07330RL
- SW1: #LCSC (none) -> C455281; Proveedor (none) -> LCSC; manf# TS-1187A-C-C-B -> TS-1088R-02526
- U1: Proveedor (none) -> RAK
- U2: #Mouser (none) -> 579-MCP1700T3302EMAY; Proveedor (none) -> Mouser; manf# (none) -> MCP1700T3302EMAY
- U3: Proveedor (none) -> Unit electronics; manf# (none) -> CP2102
- U5: value MCP73831-3-OT -> MCP73831; #LCSC (none) -> C424093; Proveedor (none) -> LCSC; manf# MCP73831T-5ACI/OT -> MCP73831T-2ACI/OT

Commit message: update cache
Parts:
- U2: symbol Regulator:MCP1700_DFN6 -> bastwan-wle-rescue:MCP1700_DFN6-Regulator
Changed lines of the file:
@@
 NoConn ~ 3950 1425
 $Comp
-L Regulator:MCP1700_DFN6 U2
+L bastwan-wle-rescue:MCP1700_DFN6-Regulator U2
 U 1 1 60F6422D
 P 2985 4295

Commit message: Change_connector
Parts:
- D4: #LCSC C72043 -> C205443; manf# 19-217/GHC-YR1S2/3T -> ORH-G36G
- D5: #LCSC C72044 -> C118330; manf# 19-217/R6C-AL1M2VY/3T -> D-060306R1/SS2/L
- J5: footprint Connector_PinHeader_2.54mm:PinHeader_1x04_P2.54mm_Vertical -> Connector:Tag-Connect_TC2030-IDC-NL_2x03_P1.27mm_Vertical; symbol Connector:Conn_01x04_Male -> Connector:Conn_01x06_Female
Connections:
- net GND: now also J5.5 (Pin_5); no longer J5.4 (Pin_4)
- net RST: now also J5.4 (Pin_4)
- no-connect marks 23 -> 24
Changed lines of the file:
@@
 F 1 "CHR" V 1693 7388 50  0000 L CNN
 F 2 "LED_SMD:LED_0603_1608Metric_Pad1.05x0.95mm_HandSolder" H 1655 7310 50  0001 C CNN
-F 3 "https://datasheet.lcsc.com/lcsc/1811101510_Everlight-Elec-19-217-GHC-YR1S2-3T_C72043.pdf" H 1655 7310 50  0001 C CNN
-F 4 "19-217/GHC-YR1S2/3T" H -235 30  50  0001 C CNN "manf#"
-F 5 "C72043" H 1655 7310 50  0001 C CNN "#LCSC"
+F 3 "https://lcsc.com/product-detail/Light-Emitting-Diodes-LED_Orient-ORH-G36G_C205443.html" H 1655 7310 50  0001 C CNN
+F 4 "ORH-G36G" H -235 30  50  0001 C CNN "manf#"
+F 5 "C205443" H 1655 7310 50  0001 C CNN "#LCSC"
 F 6 "LCSC" H 1655 7310 50  0001 C CNN "Proveedor"
 	1    1655 7310
@@
 Text Notes 3695 5655 0    79   ~ 0
 LIPO MONITORING
-Text Label 9450 4350 0    50   ~ 0
+Text Label 9785 4350 2    50   ~ 0
 SWDIO
-Text Label 9450 4450 0    50   ~ 0
+Text Label 9785 4450 2    50   ~ 0
 SWCLK
 $Comp
@@
 F 1 "D13" H 7848 4700 50  0000 C CNN
 F 2 "LED_SMD:LED_0603_1608Metric_Pad1.05x0.95mm_HandSolder" H 7855 4575 50  0001 C CNN
-F 3 "https://datasheet.lcsc.com/lcsc/1811101510_Everlight-Elec-19-217-R6C-AL1M2VY-3T_C72044.pdf" H 7855 4575 50  0001 C CNN
-F 4 "19-217/R6C-AL1M2VY/3T" H 1740 -3020 50  0001 C CNN "manf#"
-F 5 "C72044" H 7855 4575 50  0001 C CNN "#LCSC"
+F 3 "https://lcsc.com/product-detail/Light-Emitting-Diodes-LED_ARKLED-Wuxi-ARK-Tech-Elec-D-060306R1-SS2-L_C118330.html" H 7855 4575 50  0001 C CNN
+F 4 "D-060306R1/SS2/L" H 1740 -3020 50  0001 C CNN "manf#"
+F 5 "C118330" H 7855 4575 50  0001 C CNN "#LCSC"
 F 6 "LCSC" H 7855 4575 50  0001 C CNN "Proveedor"
 	1    7855 4575
@@
 	7825 6465 7825 6535
 Wire Wire Line
-	9780 4665 9780 4550
-Wire Wire Line
-	9780 4550 9450 4550
+	9780 4665 9780 4650
 Wire Wire Line
 	9780 4150 9780 4250
 Wire Wire Line
-	9780 4250 9450 4250
-$Comp
-L Connector:Conn_01x04_Male J5
+	9780 4250 9870 4250
+$Comp
+L Connector:Conn_01x06_Female J5
 U 1 1 5E1A06D2
-P 9250 4350
-F 0 "J5" H 9358 4631 50  0000 C CNN
-F 1 "SWD" H 9358 4540 50  0000 C CNN
-F 2 "Connector_PinHeader_2.54mm:PinHeader_1x04_P2.54mm_Vertical" H 9250 4350 50  0001 C CNN
-F 3 "~" H 9250 4350 50  0001 C CNN
-	1    9250 4350
+P 10070 4450
+F 0 "J5" H 10178 4731 50  0000 C CNN
+F 1 "SWD" H 10178 4640 50  0000 C CNN
+F 2 "Connector:Tag-Connect_TC2030-IDC-NL_2x03_P1.27mm_Vertical" H 10070 4450 50  0001 C CNN
+F 3 "~" H 10070 4450 50  0001 C CNN
+	1    10070 4450
 	1    0    0    -1
 $EndComp
@@
 	1    0    0    -1
 $EndComp
+Wire Wire Line
+	9870 4350 9785 4350
+Wire Wire Line
+	9785 4450 9870 4450
+Wire Wire Line
+	9870 4650 9780 4650
+NoConn ~ 9870 4750
+Text Label 9785 4550 2    50   ~ 0
+RST
+Wire Wire Line
+	9870 4550 9785 4550
 $EndSCHEMATC

Commit message: update routing v1.0
Parts:
- C1, C3, C4, C5, C6, C7: footprint Capacitor_SMD:C_0402_1005Metric_Pad0.74x0.62mm_HandSolder -> Capacitor_SMD:C_0603_1608Metric_Pad1.08x0.95mm_HandSolder
- R2, R3, R4, R6, R8, R9: footprint Resistor_SMD:R_0402_1005Metric_Pad0.72x0.64mm_HandSolder -> Resistor_SMD:R_0603_1608Metric
Other:
- moved on the sheet: C5, D4, R6, R8, U5

Commit message: Change_Cp2102_Add_USB_C
Parts:
- removed U3: CP2102N-A01-GQFN28, Package_DFN_QFN:QFN-28-1EP_5x5mm_P0.5mm_EP3.35x3.35mm, symbol Interface_USB:CP2102N-A01-GQFN28
- added C8: 0.1uF, Capacitor_SMD:C_0603_1608Metric_Pad1.08x0.95mm_HandSolder, symbol Device:C_Small
- added C9: 10uF, Capacitor_SMD:C_0603_1608Metric_Pad1.08x0.95mm_HandSolder, symbol Device:C_Small
- added R1, R5: 5.1K, Resistor_SMD:R_0603_1608Metric_Pad0.98x0.95mm_HandSolder, symbol Device:R_Small
- added U3: CP2104, Package_DFN_QFN:QFN-24-1EP_4x4mm_P0.5mm_EP2.6x2.6mm, symbol Interface_USB:CP2104
- C7: value 1uF -> 10uF; #LCSC C107372 -> C326057; manf# CL05A105KQ5NNNC -> CC0603KRX5R6BB106
- J1: value USB_B_Micro -> USB_C; footprint Connectors:U254051N4BH806 -> Connectors:C393939; symbol bastwan-wle-rescue:USB_B_Micro-Connector-Bast_WAN-rescue -> Connector:USB_C_Plug_USB2.0; #LCSC C319170 -> C393939; manf# U254-051N-4BH806 -> TYPE-C16PIN
Connections:
- net +3V3: now also U3.5 (VIO), U3.6 (VDD)
- net D+: now also J1.A6 (D+), U3.3 (D+); no longer J1.3 (D+)
- net D-: now also J1.A7 (D-), U3.4 (D-); no longer J1.2 (D-)
- net GND: now also J1.A1 (GND), J1.A12 (GND), J1.B1 (GND), J1.B12 (GND), C8.2, C9.2, R1.1, R5.1, U3.2 (GND), U3.25 (PAD); no longer J1.5 (GND), J1.6 (Shield)
- net RX_USB: now also U3.20 (RXD)
- net TX_USB: now also U3.21 (TXD)
- net VBUS: now also J1.A4 (VBUS), J1.A9 (VBUS), J1.B4 (VBUS), J1.B9 (VBUS), C8.1, U3.7 (REGIN), U3.8 (VBUS); no longer J1.1 (VBUS)
- new net: J1.A5 (CC), R1.2
- new net: J1.B5 (VCONN), R5.2
- new net: C9.1, U3.16 (VPP)
- no-connect marks 24 -> 19
Other:
- moved on the sheet: C1, C7, J4, R3, R4

Commit message: Change_BOM
Parts:
- C1, C6, C8: #LCSC C106209 -> C14663; manf# CC0402ZRY5V7BB104 -> CC0603KRX7R9BB104
- C3, C4, C5: #LCSC C15525 -> C326057
- R1, R5: #LCSC (none) -> C131715; Proveedor (none) -> LCSC; manf# (none) -> RK73B1JTTD512J
- R2: #LCSC C284273 -> C15458; manf# ARG02FTC1003 -> 0603WAJ0104T5E
- R3: #LCSC C93949 -> C304688; manf# RC0402JR-071ML -> RS-03K105JT
- R4: #LCSC C22276 -> (none); #Mouser (none) -> 667-ERJ-U03J155V; Proveedor LCSC -> Mouser; manf# 0402WGF1504TCE -> ERJ-U03J155V
- R6: #LCSC C425517 -> C384295; manf# TC0250F1001TCE -> WR06X102JTL
- R8, R9: #LCSC C105876 -> C103542; manf# RC0402JR-07330RL -> RTT033300FTP
- U3: #LCSC (none) -> C47742; Proveedor (none) -> LCSC; manf# (none) -> CP2104-F03-GMR
Changed lines of the file:
@@
 F 1 "10uF" H 2025 4360 50  0000 L CNN
 F 2 "Capacitor_SMD:C_0603_1608Metric_Pad1.08x0.95mm_HandSolder" H 2240 4435 50  0001 C CNN
-F 3 "https://datasheet.lcsc.com/lcsc/1810191215_Samsung-Electro-Mechanics-CL05A106MQ5NUNC_C15525.pdf" H 2240 4435 50  0001 C CNN
+F 3 "https://datasheet.lcsc.com/lcsc/1811031143_YAGEO-CC0603KRX5R6BB106_C326057.pdf" H 2240 4435 50  0001 C CNN
 F 4 "CL05A106MQ5NUNC" H 540 90  50  0001 C CNN "manf#"
-F 5 "C15525" H 2240 4435 50  0001 C CNN "#LCSC"
+F 5 "C326057" H 2240 4435 50  0001 C CNN "#LCSC"
 F 6 "LCSC" H 2240 4435 50  0001 C CNN "Proveedor"
 	1    2240 4435
@@
 F 1 "10uF" H 3652 4405 50  0000 L CNN
 F 2 "Capacitor_SMD:C_0603_1608Metric_Pad1.08x0.95mm_HandSolder" H 3560 4450 50  0001 C CNN
-F 3 "https://datasheet.lcsc.com/lcsc/1810191215_Samsung-Electro-Mechanics-CL05A106MQ5NUNC_C15525.pdf" H 3560 4450 50  0001 C CNN
+F 3 "https://datasheet.lcsc.com/lcsc/1811031143_YAGEO-CC0603KRX5R6BB106_C326057.pdf" H 3560 4450 50  0001 C CNN
 F 4 "CL05A106MQ5NUNC" H 540 90  50  0001 C CNN "manf#"
-F 5 "C15525" H 3560 4450 50  0001 C CNN "#LCSC"
+F 5 "C326057" H 3560 4450 50  0001 C CNN "#LCSC"
 F 6 "LCSC" H 3560 4450 50  0001 C CNN "Proveedor"
 	1    3560 4450
@@
 F 1 "10uF" H 2192 6640 50  0000 L CNN
 F 2 "Capacitor_SMD:C_0603_1608Metric_Pad1.08x0.95mm_HandSolder" H 2100 6685 50  0001 C CNN
-F 3 "https://datasheet.lcsc.com/lcsc/1810191215_Samsung-Electro-Mechanics-CL05A106MQ5NUNC_C15525.pdf" H 2100 6685 50  0001 C CNN
+F 3 "https://datasheet.lcsc.com/lcsc/1811031143_YAGEO-CC0603KRX5R6BB106_C326057.pdf" H 2100 6685 50  0001 C CNN
 F 4 "CL05A106MQ5NUNC" H -15 10  50  0001 C CNN "manf#"
-F 5 "C15525" H 2100 6685 50  0001 C CNN "#LCSC"
+F 5 "C326057" H 2100 6685 50  0001 C CNN "#LCSC"
 F 6 "LCSC" H 2100 6685 50  0001 C CNN "Proveedor"
 	1    2100 6685
@@
 F 1 "100K" V 1585 4380 50  0000 L CNN
 F 2 "Resistor_SMD:R_0603_1608Metric" H 1660 4455 50  0001 C CNN
-F 3 "https://datasheet.lcsc.com/lcsc/1810261218_Viking-Tech-ARG02FTC1003_C284273.pdf" H 1660 4455 50  0001 C CNN
-F 4 "ARG02FTC1003" H 540 90  50  0001 C CNN "manf#"
-F 5 "C284273" H 1660 4455 50  0001 C CNN "#LCSC"
+F 3 "https://datasheet.lcsc.com/lcsc/2110251730_UNI-ROYAL-Uniroyal-Elec-0603WAJ0104T5E_C15458.pdf" H 1660 4455 50  0001 C CNN
+F 4 "0603WAJ0104T5E" H 540 90  50  0001 C CNN "manf#"
+F 5 "C15458" H 1660 4455 50  0001 C CNN "#LCSC"
 F 6 "LCSC" H 1660 4455 50  0001 C CNN "Proveedor"
 	1    1660 4455
@@
 F 1 "330" H 1934 6955 50  0000 L CNN
 F 2 "Resistor_SMD:R_0603_1608Metric" H 1875 7000 50  0001 C CNN
-F 3 "https://datasheet.lcsc.com/lcsc/1810241324_YAGEO-RC0402JR-07330RL_C105876.pdf" H 1875 7000 50  0001 C CNN
-F 4 "RC0402JR-07330RL" H -15 10  50  0001 C CNN "manf#"
-F 5 "C105876" H 1875 7000 50  0001 C CNN "#LCSC"
+F 3 "https://datasheet.lcsc.com/lcsc/1810170116_RALEC-RTT033300FTP_C103542.pdfhttps://datasheet.lcsc.com/lcsc/1810170116_RALEC-RTT033300FTP_C103542.pdf" H 1875 7000 50  0001 C CNN
+F 4 "RTT033300FTP" H -15 10  50  0001 C CNN "manf#"
+F 5 "C103542" H 1875 7000 50  0001 C CNN "#LCSC"
 F 6 "LCSC" H 1875 7000 50  0001 C CNN "Proveedor"
 	1    1875 7000
@@
 F 1 "1K" V 725 6785 50  0000 C CNN
 F 2 "Resistor_SMD:R_0603_1608Metric" H 830 6785 50  0001 C CNN
-F 3 "https://datasheet.lcsc.com/lcsc/1912111437_UNI-ROYAL-Uniroyal-Elec-TC0250F1001TCE_C425517.pdf" H 830 6785 50  0001 C CNN
-F 4 "TC0250F1001TCE" H -15 10  50  0001 C CNN "manf#"
-F 5 "C425517" H 830 6785 50  0001 C CNN "#LCSC"
+F 3 "https://datasheet.lcsc.com/lcsc/1912111437_Walsin-Tech-Corp-WR06X102JTL_C384295.pdf" H 830 6785 50  0001 C CNN
+F 4 "WR06X102JTL" H -15 10  50  0001 C CNN "manf#"
+F 5 "C384295" H 830 6785 50  0001 C CNN "#LCSC"
 F 6 "LCSC" H 830 6785 50  0001 C CNN "Proveedor"
 	1    830  6785
@@
 F 1 "1M" H 3444 5955 50  0000 L CNN
 F 2 "Resistor_SMD:R_0603_1608Metric" H 3385 6000 50  0001 C CNN
-F 3 "https://datasheet.lcsc.com/lcsc/1810231331_YAGEO-RC0402JR-071ML_C93949.pdf" H 3385 6000 50  0001 C CNN
-F 4 "RC0402JR-071ML" H -2650 1235 50  0001 C CNN "manf#"
-F 5 "C93949" H 3385 6000 50  0001 C CNN "#LCSC"
+F 3 "https://datasheet.lcsc.com/lcsc/1811061728_FH-Guangdong-Fenghua-Advanced-Tech-RS-03K105JT_C304688.pdf" H 3385 6000 50  0001 C CNN
+F 4 "RS-03K105JT" H -2650 1235 50  0001 C CNN "manf#"
+F 5 "C304688" H 3385 6000 50  0001 C CNN "#LCSC"
 F 6 "LCSC" H 3385 6000 50  0001 C CNN "Proveedor"
 	1    3385 6000
@@
 F 1 "1.5M" H 3444 6320 50  0000 L CNN
 F 2 "Resistor_SMD:R_0603_1608Metric" H 3385 6365 50  0001 C CNN
-F 3 "https://datasheet.lcsc.com/lcsc/1810301422_UNI-ROYAL-Uniroyal-Elec-0402WGF1504TCE_C22276.pdf" H 3385 6365 50  0001 C CNN
-F 4 "0402WGF1504TCE" H -2650 1235 50  0001 C CNN "manf#"
-F 5 "C22276" H 3385 6365 50  0001 C CNN "#LCSC"
-F 6 "LCSC" H 3385 6365 50  0001 C CNN "Proveedor"
+F 3 "https://www.mouser.mx/datasheet/2/315/AOA0000C334-1314047.pdf" H 3385 6365 50  0001 C CNN
+F 4 "ERJ-U03J155V" H -2650 1235 50  0001 C CNN "manf#"
+F 5 "" H 3385 6365 50  0001 C CNN "#LCSC"
+F 6 "Mouser" H 3385 6365 50  0001 C CNN "Proveedor"
+F 7 "667-ERJ-U03J155V" H 3385 6365 50  0001 C CNN "#Mouser"
 	1    3385 6365
 	1    0    0    -1
@@
 F 1 "330" V 7405 4575 50  0000 C CNN
 F 2 "Resistor_SMD:R_0603_1608Metric" H 7510 4575 50  0001 C CNN
-F 3 "https://datasheet.lcsc.com/lcsc/1810241324_YAGEO-RC0402JR-07330RL_C105876.pdf" H 7510 4575 50  0001 C CNN
-F 4 "RC0402JR-07330RL" H 1740 -3020 50  0001 C CNN "manf#"
-F 5 "C105876" H 7510 4575 50  0001 C CNN "#LCSC"
+F 3 "https://datasheet.lcsc.com/lcsc/1810170116_RALEC-RTT033300FTP_C103542.pdfhttps://datasheet.lcsc.com/lcsc/1810170116_RALEC-RTT033300FTP_C103542.pdf" H 7510 4575 50  0001 C CNN
+F 4 "RTT033300FTP" H 1740 -3020 50  0001 C CNN "manf#"
+F 5 "C103542" H 7510 4575 50  0001 C CNN "#LCSC"
 F 6 "LCSC" H 7510 4575 50  0001 C CNN "Proveedor"
 	1    7510 4575
@@
 F 1 "0.1uF" H 9392 2035 50  0000 L CNN
 F 2 "Capacitor_SMD:C_0603_1608Metric_Pad1.08x0.95mm_HandSolder" H 9300 2080 50  0001 C CNN
-F 3 "https://datasheet.lcsc.com/lcsc/1810241334_YAGEO-CC0402ZRY5V7BB104_C106209.pdf" H 9300 2080 50  0001 C CNN
-F 4 "C106209" H 9300 2080 50  0001 C CNN "#LCSC"
+F 3 "https://datasheet.lcsc.com/lcsc/1809301912_YAGEO-CC0603KRX7R9BB104_C14663.pdf" H 9300 2080 50  0001 C CNN
+F 4 "C14663" H 9300 2080 50  0001 C CNN "#LCSC"
 F 5 "LCSC" H 9300 2080 50  0001 C CNN "Proveedor"
-F 6 "CC0402ZRY5V7BB104" H 9300 2080 50  0001 C CNN "manf#"
+F 6 "CC0603KRX7R9BB104" H 9300 2080 50  0001 C CNN "manf#"
 	1    9300 2080
 	1    0    0    -1
@@
 F 1 "CP2104" H 4965 4405 50  0000 C CNN
 F 2 "Package_DFN_QFN:QFN-24-1EP_4x4mm_P0.5mm_EP2.6x2.6mm" H 5705 4470 50  0001 L CNN
-F 3 "https://www.mouser.mx/datasheet/2/368/cp2104-1397921.pdf" H 5005 6670 50  0001 C CNN
+F 3 "https://datasheet.lcsc.com/lcsc/1809191938_SILICON-LABS-CP2104-F03-GMR_C47742.pdf" H 5005 6670 50  0001 C CNN
+F 4 "C47742" H 5555 5420 50  0001 C CNN "#LCSC"
+F 5 "LCSC" H 5555 5420 50  0001 C CNN "Proveedor"
+F 6 "CP2104-F03-GMR" H 5555 5420 50  0001 C CNN "manf#"
 	1    5555 5420
 	1    0    0    -1
@@
 F 1 "0.1uF" H 6522 4455 50  0000 L CNN
 F 2 "Capacitor_SMD:C_0603_1608Metric_Pad1.08x0.95mm_HandSolder" H 6430 4500 50  0001 C CNN
-F 3 "https://datasheet.lcsc.com/lcsc/1810241334_YAGEO-CC0402ZRY5V7BB104_C106209.pdf" H 6430 4500 50  0001 C CNN
-F 4 "C106209" H 6430 4500 50  0001 C CNN "#LCSC"
+F 3 "https://datasheet.lcsc.com/lcsc/1809301912_YAGEO-CC0603KRX7R9BB104_C14663.pdf" H 6430 4500 50  0001 C CNN
+F 4 "C14663" H 6430 4500 50  0001 C CNN "#LCSC"
 F 5 "LCSC" H 6430 4500 50  0001 C CNN "Proveedor"
-F 6 "CC0402ZRY5V7BB104" H 6430 4500 50  0001 C CNN "manf#"
+F 6 "CC0603KRX7R9BB104" H 6430 4500 50  0001 C CNN "manf#"
 	1    6430 4500
 	1    0    0    -1
@@
 F 1 "0.1uF" H 4782 5145 50  0000 L CNN
 F 2 "Capacitor_SMD:C_0603_1608Metric_Pad1.08x0.95mm_HandSolder" H 4690 5190 50  0001 C CNN
-F 3 "https://datasheet.lcsc.com/lcsc/1810241334_YAGEO-CC0402ZRY5V7BB104_C106209.pdf" H 4690 5190 50  0001 C CNN
-F 4 "C106209" H 4690 5190 50  0001 C CNN "#LCSC"
+F 3 "https://datasheet.lcsc.com/lcsc/1809301912_YAGEO-CC0603KRX7R9BB104_C14663.pdf" H 4690 5190 50  0001 C CNN
+F 4 "C14663" H 4690 5190 50  0001 C CNN "#LCSC"
 F 5 "LCSC" H 4690 5190 50  0001 C CNN "Proveedor"
-F 6 "CC0402ZRY5V7BB104" H 4690 5190 50  0001 C CNN "manf#"
+F 6 "CC0603KRX7R9BB104" H 4690 5190 50  0001 C CNN "manf#"
 	1    4690 5190
 	1    0    0    -1
@@
 F 1 "5.1K" V 1650 1165 50  0000 C CNN
 F 2 "Resistor_SMD:R_0603_1608Metric_Pad0.98x0.95mm_HandSolder" H 1725 1010 50  0001 C CNN
-F 3 "~" H 1725 1010 50  0001 C CNN
+F 3 "https://datasheet.lcsc.com/lcsc/1811031511_KOA-Speer-Elec-RK73B1JTTD512J_C131715.pdf" H 1725 1010 50  0001 C CNN
+F 4 "C131715" H 1725 1010 50  0001 C CNN "#LCSC"
+F 5 "LCSC" H 1725 1010 50  0001 C CNN "Proveedor"
+F 6 "RK73B1JTTD512J" H 1725 1010 50  0001 C CNN "manf#"
 	1    1725 1010
 	0    1    1    0
@@
 F 1 "5.1K" V 1680 1290 50  0000 C CNN
 F 2 "Resistor_SMD:R_0603_1608Metric_Pad0.98x0.95mm_HandSolder" H 1725 1110 50  0001 C CNN
-F 3 "~" H 1725 1110 50  0001 C CNN
+F 3 "https://datasheet.lcsc.com/lcsc/1811031511_KOA-Speer-Elec-RK73B1JTTD512J_C131715.pdf" H 1725 1110 50  0001 C CNN
+F 4 "C131715" H 1725 1110 50  0001 C CNN "#LCSC"
+F 5 "LCSC" H 1725 1110 50  0001 C CNN "Proveedor"
+F 6 "RK73B1JTTD512J" H 1725 1110 50  0001 C CNN "manf#"
 	1    1725 1110
 	0    1    1    0
